File: PCB/hackpad-v2.kicad_pcb (KiCad board)
At the start: 2 copper layers, 95 x 75 mm, 24 parts, among them SW1 RotaryEncoder, SW2 SW_Push, SW3 SW_Push, SW4 SW_Push, U1 XIAO-RP2040-DIP

Commit message: some more blender stuff
Parts:
- D1, D10, D11, D12, D13, D14, D2, D3, D4, D5, D6, D7, D8, D9: footprint LED_SMD:LED_SK6812MINI_PLCC4_3.5x3.5mm_P1.75mm -> kai's library:LED_SK6812MINI_PLCC4_3.5x3.5mm_P1.75mm
