File: PCB/hackpad-v2.kicad_sch (KiCad schematic)
At the start: 19 parts, among them SW1 RotaryEncoder, SW2 SW_Push, SW3 SW_Push, SW4 SW_Push, U1 XIAO-RP2040-DIP

Commit message: some more blender stuff
Parts:
- D1, D10, D11, D12, D13, D14, D2, D3, D4, D5, D6, D7, D8, D9: footprint LED_SMD:LED_SK6812MINI_PLCC4_3.5x3.5mm_P1.75mm -> kai's library:LED_SK6812MINI_PLCC4_3.5x3.5mm_P1.75mm
Changed lines of the file:
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@@
 			)
 		)
-		(property "Footprint" "LED_SMD:LED_SK6812MINI_PLCC4_3.5x3.5mm_P1.75mm"
+		(property "Footprint" "kai's library:LED_SK6812MINI_PLCC4_3.5x3.5mm_P1.75mm"
 			(at 173.99 67.31 0)
 			(effects
@@
 			)
 		)
-		(property "Footprint" "LED_SMD:LED_SK6812MINI_PLCC4_3.5x3.5mm_P1.75mm"
+		(property "Footprint" "kai's library:LED_SK6812MINI_PLCC4_3.5x3.5mm_P1.75mm"
 			(at 97.79 44.45 0)
 			(effects
@@
 			)
 		)
-		(property "Footprint" "LED_SMD:LED_SK6812MINI_PLCC4_3.5x3.5mm_P1.75mm"
+		(property "Footprint" "kai's library:LED_SK6812MINI_PLCC4_3.5x3.5mm_P1.75mm"
 			(at 158.75 44.45 0)
 			(effects
@@
 			)
 		)
-		(property "Footprint" "LED_SMD:LED_SK6812MINI_PLCC4_3.5x3.5mm_P1.75mm"
+		(property "Footprint" "kai's library:LED_SK6812MINI_PLCC4_3.5x3.5mm_P1.75mm"
 			(at 128.27 44.45 0)
 			(effects
@@
 			)
 		)
-		(property "Footprint" "LED_SMD:LED_SK6812MINI_PLCC4_3.5x3.5mm_P1.75mm"
+		(property "Footprint" "kai's library:LED_SK6812MINI_PLCC4_3.5x3.5mm_P1.75mm"
 			(at 143.51 44.45 0)
 			(effects
@@
 			)
 		)
-		(property "Footprint" "LED_SMD:LED_SK6812MINI_PLCC4_3.5x3.5mm_P1.75mm"
+		(property "Footprint" "kai's library:LED_SK6812MINI_PLCC4_3.5x3.5mm_P1.75mm"
 			(at 128.27 67.31 0)
 			(effects
@@
 			)
 		)
-		(property "Footprint" "LED_SMD:LED_SK6812MINI_PLCC4_3.5x3.5mm_P1.75mm"
+		(property "Footprint" "kai's library:LED_SK6812MINI_PLCC4_3.5x3.5mm_P1.75mm"
 			(at 189.23 44.45 0)
 			(effects
@@
 			)
 		)
-		(property "Footprint" "LED_SMD:LED_SK6812MINI_PLCC4_3.5x3.5mm_P1.75mm"
+		(property "Footprint" "kai's library:LED_SK6812MINI_PLCC4_3.5x3.5mm_P1.75mm"
 			(at 113.03 44.45 0)
 			(effects
@@
 			)
 		)
-		(property "Footprint" "LED_SMD:LED_SK6812MINI_PLCC4_3.5x3.5mm_P1.75mm"
+		(property "Footprint" "kai's library:LED_SK6812MINI_PLCC4_3.5x3.5mm_P1.75mm"
 			(at 204.47 44.45 0)
 			(effects
@@
 			)
 		)
-		(property "Footprint" "LED_SMD:LED_SK6812MINI_PLCC4_3.5x3.5mm_P1.75mm"
+		(property "Footprint" "kai's library:LED_SK6812MINI_PLCC4_3.5x3.5mm_P1.75mm"
 			(at 158.75 67.31 0)
 			(effects
@@
 			)
 		)
-		(property "Footprint" "LED_SMD:LED_SK6812MINI_PLCC4_3.5x3.5mm_P1.75mm"
+		(property "Footprint" "kai's library:LED_SK6812MINI_PLCC4_3.5x3.5mm_P1.75mm"
 			(at 97.79 67.31 0)
 			(effects
@@
 			)
 		)
-		(property "Footprint" "LED_SMD:LED_SK6812MINI_PLCC4_3.5x3.5mm_P1.75mm"
+		(property "Footprint" "kai's library:LED_SK6812MINI_PLCC4_3.5x3.5mm_P1.75mm"
 			(at 113.03 67.31 0)
 			(effects
@@
 			)
 		)
-		(property "Footprint" "LED_SMD:LED_SK6812MINI_PLCC4_3.5x3.5mm_P1.75mm"
+		(property "Footprint" "kai's library:LED_SK6812MINI_PLCC4_3.5x3.5mm_P1.75mm"
 			(at 173.99 44.45 0)
 			(effects
@@
 			)
 		)
-		(property "Footprint" "LED_SMD:LED_SK6812MINI_PLCC4_3.5x3.5mm_P1.75mm"
+		(property "Footprint" "kai's library:LED_SK6812MINI_PLCC4_3.5x3.5mm_P1.75mm"
 			(at 143.51 67.31 0)
 			(effects
